Commit message: improvements based on testin

File: industrial_extrinsic_cal/urdf/camera_scene.urdf (robot description, URDF)
Before this commit: robot industrial_kinect_calibration, 15 links, 14 joints
Links:
- removed link kinect_frame
- removed link kinect_ir_link
- removed link kinect_ir_optical_frame
- removed link kinect_link
- removed link kinect_link_pitch
- removed link kinect_link_x_trans
- removed link kinect_link_y_trans
- removed link kinect_link_yaw
- removed link kinect_link_z_trans
- removed link kinect_rgb_frame
- removed link kinect_rgb_link
- removed link kinect_rgb_optical_frame
- added link camera_frame; collision box size=0.04 0.22 0.04; visual box size=0.04 0.22 0.04
- added link camera_ir_link; visual sphere radius=0.0005
- added link camera_ir_optical_frame
- added link camera_link
- added link camera_link_pitch
- added link camera_link_x_trans; visual sphere radius=0.0005
- added link camera_link_y_trans
- added link camera_link_yaw
- added link camera_link_z_trans
- added link camera_rgb_frame
- added link camera_rgb_link; visual sphere radius=0.0005
- added link camera_rgb_optical_frame
Joints:
- removed joint kinect_frame_joint
- removed joint kinect_ir_joint
- removed joint kinect_ir_optical_frame_joint
- removed joint kinect_link_pitch_joint
- removed joint kinect_link_roll_joint
- removed joint kinect_link_x_joint
- removed joint kinect_link_y_joint
- removed joint kinect_link_yaw_joint
- removed joint kinect_link_z_joint
- removed joint kinect_rgb_frame_joint
- removed joint kinect_rgb_joint
- removed joint kinect_rgb_optical_frame_joint
- added joint camera_frame_joint: type fixed, parent camera_link, child camera_frame, origin xyz=0 0 0 rpy=0 0 0
- added joint camera_ir_joint: type fixed, parent camera_frame, child camera_ir_link, origin xyz=0 0 0 rpy=0 0 0
- added joint camera_ir_optical_frame_joint: type fixed, parent camera_ir_link, child camera_ir_optical_frame, origin xyz=0 0 0 rpy=-1.57 0 -1.57
- added joint camera_link_pitch_joint: type revolute, parent camera_link_yaw, child camera_link_pitch, origin xyz=0 0 0 rpy=0 0 0, axis 0 1 0, limit lower=-6.2832 upper=6.2832 effort=2 velocity=10
- added joint camera_link_roll_joint: type revolute, parent camera_link_pitch, child camera_link, origin xyz=0 0 0 rpy=0 0 0, axis 1 0 0, limit lower=-6.2832 upper=6.2832 effort=2 velocity=10
- added joint camera_link_x_joint: type prismatic, parent world, child camera_link_x_trans, origin xyz=0 0 0 rpy=0 0 0, axis 1 0 0, limit lower=-1.0 upper=1.0 effort=30 velocity=0.0508
- added joint camera_link_y_joint: type prismatic, parent camera_link_x_trans, child camera_link_y_trans, origin xyz=0 0 0 rpy=0 0 0, axis 0 1 0, limit lower=-1.0 upper=1.0 effort=30 velocity=0.0508
- added joint camera_link_yaw_joint: type revolute, parent camera_link_z_trans, child camera_link_yaw, origin xyz=0 0 0 rpy=0 0 0, axis 0 0 1, limit lower=-6.2832 upper=6.2832 effort=2 velocity=10
- added joint camera_link_z_joint: type prismatic, parent camera_link_y_trans, child camera_link_z_trans, origin xyz=0 0 0 rpy=0 0 0, axis 0 0 1, limit lower=-1.0 upper=1.0 effort=30 velocity=0.0508
- added joint camera_rgb_frame_joint: type fixed, parent camera_rgb_optical_frame, child camera_rgb_frame, origin xyz=0 0.0 0 rpy=0 0 0
- added joint camera_rgb_joint: type fixed, parent camera_ir_link, child camera_rgb_link, origin xyz=0 -0.03 0 rpy=0 0 0
- added joint camera_rgb_optical_frame_joint: type fixed, parent camera_rgb_link, child camera_rgb_optical_frame, origin xyz=0 0 0 rpy=-1.57 0 -1.57

File: rgbd_depth_correction/urdf/camera_scene.urdf (robot description, URDF)
Before this commit: robot industrial_kinect_calibration, 14 links, 13 joints
Links:
- removed link kinect_frame
- removed link kinect_ir_link
- removed link kinect_ir_optical_frame
- removed link kinect_link
- removed link kinect_link_pitch
- removed link kinect_link_x_trans
- removed link kinect_link_y_trans
- removed link kinect_link_yaw
- removed link kinect_link_z_trans
- removed link kinect_rgb_frame
- removed link kinect_rgb_link
- removed link kinect_rgb_optical_frame
- added link camera_frame; collision box size=0.04 0.22 0.04; visual box size=0.04 0.22 0.04
- added link camera_ir_link; visual sphere radius=0.0005
- added link camera_ir_optical_frame
- added link camera_link
- added link camera_link_pitch
- added link camera_link_x_trans; visual sphere radius=0.0005
- added link camera_link_y_trans
- added link camera_link_yaw
- added link camera_link_z_trans
- added link camera_rgb_frame
- added link camera_rgb_link; visual sphere radius=0.0005
- added link camera_rgb_optical_frame
Joints:
- removed joint kinect_frame_joint
- removed joint kinect_ir_joint
- removed joint kinect_ir_optical_frame_joint
- removed joint kinect_link_pitch_joint
- removed joint kinect_link_roll_joint
- removed joint kinect_link_x_joint
- removed joint kinect_link_y_joint
- removed joint kinect_link_yaw_joint
- removed joint kinect_link_z_joint
- removed joint kinect_rgb_frame_joint
- removed joint kinect_rgb_joint
- removed joint kinect_rgb_optical_frame_joint
- added joint camera_frame_joint: type fixed, parent camera_link, child camera_frame, origin xyz=0 0 0 rpy=0 0 0
- added joint camera_ir_joint: type fixed, parent camera_frame, child camera_ir_link, origin xyz=0 0 0 rpy=0 0 0
- added joint camera_ir_optical_frame_joint: type fixed, parent camera_ir_link, child camera_ir_optical_frame, origin xyz=0 0 0 rpy=-1.57 0 -1.57
- added joint camera_link_pitch_joint: type revolute, parent camera_link_yaw, child camera_link_pitch, origin xyz=0 0 0 rpy=0 0 0, axis 0 1 0, limit lower=-3.1415 upper=3.1415 effort=2 velocity=10
- added joint camera_link_roll_joint: type revolute, parent camera_link_pitch, child camera_link, origin xyz=0 0 0 rpy=0 0 0, axis 1 0 0, limit lower=-3.1415 upper=3.1415 effort=2 velocity=10
- added joint camera_link_x_joint: type prismatic, parent world, child camera_link_x_trans, origin xyz=0 0 0 rpy=0 0 0, axis 1 0 0, limit lower=-1.0 upper=1.0 effort=30 velocity=0.0508
- added joint camera_link_y_joint: type prismatic, parent camera_link_x_trans, child camera_link_y_trans, origin xyz=0 0 0 rpy=0 0 0, axis 0 1 0, limit lower=-1.0 upper=1.0 effort=30 velocity=0.0508
- added joint camera_link_yaw_joint: type revolute, parent camera_link_z_trans, child camera_link_yaw, origin xyz=0 0 0 rpy=0 0 0, axis 0 0 1, limit lower=-3.1415 upper=3.1415 effort=2 velocity=10
- added joint camera_link_z_joint: type prismatic, parent camera_link_y_trans, child camera_link_z_trans, origin xyz=0 0 0 rpy=0 0 0, axis 0 0 1, limit lower=-1.0 upper=1.0 effort=30 velocity=0.0508
- added joint camera_rgb_frame_joint: type fixed, parent camera_rgb_optical_frame, child camera_rgb_frame, origin xyz=0 0.0 0 rpy=0 0 0
- added joint camera_rgb_joint: type fixed, parent camera_ir_link, child camera_rgb_link, origin xyz=0 -0.03 0 rpy=0 0 0
- added joint camera_rgb_optical_frame_joint: type fixed, parent camera_rgb_link, child camera_rgb_optical_frame, origin xyz=0 0 0 rpy=-1.57 0 -1.57
